Commit message: Updated URDF

File: urdf/sentry.xacro (robot description, xacro)
@@ -71,8 +71,30 @@
   </collision>
 </link>
+<!-- Left Motor Link -->
+<link name="left_motor">
+  <inertial>
+    <origin rpy="0 0 0" xyz="0 0 0"/>
+    <mass value="1"/>
+    <inertia ixx="0.001218" ixy="0.0" ixz="0.0" iyy="0.000635" iyz="0.0" izz="0.000635"/>
+  </inertial>
+  <visual>
+    <origin rpy="0 0 0" xyz="0 0 0"/>
+    <geometry>
+      <mesh filename="package://sentry_description/meshes/motor.stl" scale="0.001 0.001 0.001"/>
+    </geometry>
+    <material name="silver"/>
+  </visual>
+  <collision>
+    <origin rpy="0 0 0" xyz="0 0 0"/>
+    <geometry>
+      <mesh filename="package://sentry_description/meshes/motor.stl" scale="0.001 0.001 0.001"/>
+    </geometry>
+  </collision>
+</link>
+<!-- JOINTS -->
+<!-- The origin of the joint is used as the origin of that component, when positioning above -->
 <!-- Joint between Left wheel and Base Link -->
-<!-- The origin of the joint is used as the origin of that component, when positioning above -->
 <joint name="left_wheel_joint" type="continuous">
-  <origin rpy="0 0 0" xyz="-0.18650 0 0.07260"/>
+  <origin rpy="0 0 0" xyz="-0.18650 0 0.11460"/>
   <parent link="base_link"/>
   <child link="left_wheel"/>
@@ -81,6 +103,7 @@
   <joint_properties damping="1.0" friction="1.0"/>
 </joint>
+<!-- Joint between right wheel and Base Link -->
 <joint name="right_wheel_joint" type="continuous">
-  <origin rpy="0 0 0" xyz="0.18650 0 0.07260"/>
+  <origin rpy="0 0 0" xyz="0.18650 0 0.11460"/>
   <parent link="base_link"/>
   <child link="right_wheel"/>
@@ -89,3 +112,9 @@
   <joint_properties damping="1.0" friction="1.0"/>
 </joint>
+<!-- Joint between Left motor and Base Link -->
+<joint name="left_motor_base_joint" type="fixed">
+  <origin rpy="0 0 0" xyz="-0.80779 0.92779 0.93831"/>
+  <parent link="base_link"/>
+  <child link="left_motor"/>
+</joint>
 </robot>

Commit message: Changed mesh URIs in sentry xacro

File: urdf/sentry.xacro (robot description, xacro)
@@ -16,5 +16,5 @@
     <origin rpy="0 0 0" xyz="0 0 0"/>
     <geometry>
-      <mesh filename="package://sentry_description/meshes/base_link.stl" scale="0.001 0.001 0.001"/>
+      <mesh filename="package://sentry_description/CAD/parts/base_link/base_link.stl" scale="0.001 0.001 0.001"/>
     </geometry>
     <material name="silver"/>
@@ -23,5 +23,5 @@
     <origin rpy="0 0 0" xyz="0 0 0"/>
     <geometry>
-      <mesh filename="package://sentry_description/meshes/base_link.stl" scale="0.001 0.001 0.001"/>
+      <mesh filename="package://sentry_description/CAD/parts/base_link/base_link.stl" scale="0.001 0.001 0.001"/>
     </geometry>
   </collision>
@@ -39,5 +39,5 @@
     <origin rpy="0 0 0" xyz="0 0 0"/>
     <geometry>
-      <mesh filename="package://sentry_description/meshes/wheel.stl" scale="0.001 0.001 0.001"/>
+      <mesh filename="package://sentry_description/CAD/parts/wheel/wheel.stl" scale="0.001 0.001 0.001"/>
     </geometry>
     <material name="silver"/>
@@ -46,5 +46,5 @@
     <origin rpy="0 0 0" xyz="0 0 0"/>
     <geometry>
-      <mesh filename="package://sentry_description/meshes/wheel.stl" scale="0.001 0.001 0.001"/>
+      <mesh filename="package://sentry_description/CAD/parts/wheel/wheel.stl" scale="0.001 0.001 0.001"/>
     </geometry>
   </collision>
@@ -60,5 +60,5 @@
     <origin rpy="0 0 0" xyz="0 0 0"/>
     <geometry>
-      <mesh filename="package://sentry_description/meshes/wheel.stl" scale="0.001 0.001 0.001"/>
+      <mesh filename="package://sentry_description/CAD/parts/wheel/wheel.stl" scale="0.001 0.001 0.001"/>
     </geometry>
     <material name="silver"/>
@@ -67,26 +67,5 @@
     <origin rpy="0 0 0" xyz="0 0 0"/>
     <geometry>
-      <mesh filename="package://sentry_description/meshes/wheel.stl" scale="0.001 0.001 0.001"/>
-    </geometry>
-  </collision>
-</link>
-<!-- Left Motor Link -->
-<link name="left_motor">
-  <inertial>
-    <origin rpy="0 0 0" xyz="0 0 0"/>
-    <mass value="1"/>
-    <inertia ixx="0.001218" ixy="0.0" ixz="0.0" iyy="0.000635" iyz="0.0" izz="0.000635"/>
-  </inertial>
-  <visual>
-    <origin rpy="0 0 0" xyz="0 0 0"/>
-    <geometry>
-      <mesh filename="package://sentry_description/meshes/motor.stl" scale="0.001 0.001 0.001"/>
-    </geometry>
-    <material name="silver"/>
-  </visual>
-  <collision>
-    <origin rpy="0 0 0" xyz="0 0 0"/>
-    <geometry>
-      <mesh filename="package://sentry_description/meshes/motor.stl" scale="0.001 0.001 0.001"/>
+      <mesh filename="package://sentry_description/CAD/parts/wheel/wheel.stl" scale="0.001 0.001 0.001"/>
     </geometry>
   </collision>
@@ -96,5 +75,5 @@
 <!-- Joint between Left wheel and Base Link -->
 <joint name="left_wheel_joint" type="continuous">
-  <origin rpy="0 0 0" xyz="-0.18650 0 0.11460"/>
+  <origin rpy="0 0 0" xyz="-0.18650 0 0.114"/>
   <parent link="base_link"/>
   <child link="left_wheel"/>
@@ -105,16 +84,11 @@
 <!-- Joint between right wheel and Base Link -->
 <joint name="right_wheel_joint" type="continuous">
-  <origin rpy="0 0 0" xyz="0.18650 0 0.11460"/>
+<!-- yaw set to 3.14159 to flip the wheel and align it properly-->
+  <origin rpy="0 0 3.14159" xyz="0.18650 0 0.114"/>
   <parent link="base_link"/>
   <child link="right_wheel"/>
-  <axis xyz="1.0 0.0 0.0"/>
+  <axis xyz="-1.0 0.0 0.0"/>
   <limit effort="10000" velocity="1000"/>
   <joint_properties damping="1.0" friction="1.0"/>
 </joint>
-<!-- Joint between Left motor and Base Link -->
-<joint name="left_motor_base_joint" type="fixed">
-  <origin rpy="0 0 0" xyz="-0.80779 0.92779 0.93831"/>
-  <parent link="base_link"/>
-  <child link="left_motor"/>
-</joint>
 </robot>

Commit message: Update sentry.xacro

File: urdf/sentry.xacro (robot description, xacro)
@@ -16,5 +16,5 @@
     <origin rpy="0 0 0" xyz="0 0 0"/>
     <geometry>
-      <mesh filename="package://sentry_description/CAD/parts/base_link/base_link.stl" scale="0.001 0.001 0.001"/>
+      <mesh filename="package://sentry_description/CAD/parts/base_link/base_link_v3.stl" scale="0.001 0.001 0.001"/>
     </geometry>
     <material name="silver"/>
@@ -23,5 +23,5 @@
     <origin rpy="0 0 0" xyz="0 0 0"/>
     <geometry>
-      <mesh filename="package://sentry_description/CAD/parts/base_link/base_link.stl" scale="0.001 0.001 0.001"/>
+      <mesh filename="package://sentry_description/CAD/parts/base_link/base_link_v3.stl" scale="0.001 0.001 0.001"/>
     </geometry>
   </collision>

Commit message: Adding new base_link

File: urdf/sentry.xacro (robot description, xacro)
@@ -16,5 +16,5 @@
     <origin rpy="0 0 0" xyz="0 0 0"/>
     <geometry>
-      <mesh filename="package://sentry_description/CAD/parts/base_link/base_link_v3.stl" scale="0.001 0.001 0.001"/>
+      <mesh filename="package://sentry_description/CAD/parts/base_link/base_link_v4.stl" scale="0.001 0.001 0.001"/>
     </geometry>
     <material name="silver"/>
@@ -23,5 +23,5 @@
     <origin rpy="0 0 0" xyz="0 0 0"/>
     <geometry>
-      <mesh filename="package://sentry_description/CAD/parts/base_link/base_link_v3.stl" scale="0.001 0.001 0.001"/>
+      <mesh filename="package://sentry_description/CAD/parts/base_link/base_link_v4.stl" scale="0.001 0.001 0.001"/>
     </geometry>
   </collision>

Commit message: Adding lidar

File: urdf/sentry.xacro (robot description, xacro)
@@ -71,4 +71,25 @@
   </collision>
 </link>
+<link name="laser_sensor">
+  <inertial>
+    <!--<origin rpy="0 0 0" xyz="0.16605823931257102 -0.20000099435655025 0.0635739775901992"/>-->
+    <origin rpy="0 0 0" xyz="0 0 0"/>
+    <mass value="1"/>
+    <inertia ixx="0.001218" ixy="0.0" ixz="0.0" iyy="0.000635" iyz="0.0" izz="0.000635"/>
+  </inertial>
+  <visual>
+    <origin rpy="0 0 0" xyz="0 0 0"/>
+    <geometry>
+      <mesh filename="package://sentry_description/CAD/parts/Lidar/ydlidar_x4 v2.stl" scale="0.001 0.001 0.001"/>
+    </geometry>
+    <material name="silver"/>
+  </visual>
+  <collision>
+    <origin rpy="0 0 0" xyz="0 0 0"/>
+    <geometry>
+      <mesh filename="package://sentry_description/CAD/parts/Lidar/ydlidar_x4 v2.stl" scale="0.001 0.001 0.001"/>
+    </geometry>
+  </collision>
+</link>
 <!-- JOINTS -->
 <!-- The origin of the joint is used as the origin of that component, when positioning above -->

Commit message: Adding lidar joint

File: urdf/sentry.xacro (robot description, xacro)
@@ -113,3 +113,8 @@
   <joint_properties damping="1.0" friction="1.0"/>
 </joint>
+<joint name="lidar_joint" type="fixed">
+    <parent link="base_link"/>
+    <child link="laser_sensor"/>
+    <origin rpy= "0 0 0" xyz="0 0 "/>
+  </joint>
 </robot>

Commit message: Fixing lidar origin

File: urdf/sentry.xacro (robot description, xacro)
@@ -116,5 +116,5 @@
     <parent link="base_link"/>
     <child link="laser_sensor"/>
-    <origin rpy= "0 0 0" xyz="0 0 "/>
+    <origin rpy= "0 0 0" xyz="0 0 0.17"/>
   </joint>
 </robot>

Commit message: hanging origin values

File: urdf/sentry.xacro (robot description, xacro)
@@ -116,5 +116,5 @@
     <parent link="base_link"/>
     <child link="laser_sensor"/>
-    <origin rpy= "0 0 0" xyz="0 0 0.17"/>
+    <origin rpy= "0 0 0" xyz="0 0 1.5"/>
   </joint>
 </robot>

Commit message: Fixing lidar orientation

File: urdf/sentry.xacro (robot description, xacro)
@@ -116,5 +116,5 @@
     <parent link="base_link"/>
     <child link="laser_sensor"/>
-    <origin rpy= "0 0 0" xyz="0 0 1.5"/>
+    <origin rpy= "0 0 0" xyz="0 -0.22 1.5"/>
   </joint>
 </robot>

Commit message: Update sentry.xacro

File: urdf/sentry.xacro (robot description, xacro)
@@ -7,4 +7,6 @@
 <!--  Base link -->
 <!-- Combine as much bodies as possible into the base_link, this will reduce the complexity of the design -->
+<link name="dummy">
+   </link>
 <link name="base_link">
   <inertial>
@@ -37,5 +39,5 @@
   </inertial>
   <visual>
-    <origin rpy="0 0 0" xyz="0 0 0"/>
+    <origin rpy="0 0 0" xyz="-0.18650 0 0.114"/>
     <geometry>
       <mesh filename="package://sentry_description/CAD/parts/wheel/wheel.stl" scale="0.001 0.001 0.001"/>
@@ -58,5 +60,5 @@
   </inertial>
   <visual>
-    <origin rpy="0 0 0" xyz="0 0 0"/>
+    <origin rpy="0 0 3.14159" xyz="0.18650 0 0.114"/>
     <geometry>
       <mesh filename="package://sentry_description/CAD/parts/wheel/wheel.stl" scale="0.001 0.001 0.001"/>
@@ -75,9 +77,9 @@
     <!--<origin rpy="0 0 0" xyz="0.16605823931257102 -0.20000099435655025 0.0635739775901992"/>-->
     <origin rpy="0 0 0" xyz="0 0 0"/>
-    <mass value="1"/>
+    <mass value="0.5"/>
     <inertia ixx="0.001218" ixy="0.0" ixz="0.0" iyy="0.000635" iyz="0.0" izz="0.000635"/>
   </inertial>
   <visual>
-    <origin rpy="0 0 0" xyz="0 0 0"/>
+    <origin rpy= "0 0 0" xyz="0 0.22 1.5"/>
     <geometry>
       <mesh filename="package://sentry_description/CAD/parts/Lidar/ydlidar_x4 v2.stl" scale="0.001 0.001 0.001"/>
@@ -115,6 +117,10 @@
 <joint name="lidar_joint" type="fixed">
     <parent link="base_link"/>
-    <child link="laser_sensor"/>
-    <origin rpy= "0 0 0" xyz="0 -0.22 1.5"/>
-  </joint>
+    <child link="laser_sensor"/>s
+    <origin rpy= "0 0 0" xyz="0 0.22 1.5"/>
+</joint>
+<joint name="dummy_joint" type="fixed">
+    <parent link="dummy"/>
+    <child link="base_link"/>
+</joint>
 </robot>

Commit message: Updating mesh files

File: urdf/sentry.xacro (robot description, xacro)
@@ -18,5 +18,5 @@
     <origin rpy="0 0 0" xyz="0 0 0"/>
     <geometry>
-      <mesh filename="package://sentry_description/CAD/parts/base_link/base_link_v4.stl" scale="0.001 0.001 0.001"/>
+      <mesh filename="package://sentry_description/CAD/parts/base-link/base_link_no wheels v2.stl" scale="0.001 0.001 0.001"/>
     </geometry>
     <material name="silver"/>
@@ -25,5 +25,5 @@
     <origin rpy="0 0 0" xyz="0 0 0"/>
     <geometry>
-      <mesh filename="package://sentry_description/CAD/parts/base_link/base_link_v4.stl" scale="0.001 0.001 0.001"/>
+      <mesh filename="package://sentry_description/CAD/parts/base-link/base_link_no wheels v2.stl" scale="0.001 0.001 0.001"/>
     </geometry>
   </collision>
@@ -41,5 +41,5 @@
     <origin rpy="0 0 0" xyz="-0.18650 0 0.114"/>
     <geometry>
-      <mesh filename="package://sentry_description/CAD/parts/wheel/wheel.stl" scale="0.001 0.001 0.001"/>
+      <mesh filename="package://sentry_description/CAD/parts/wheel/wheel v3.stl" scale="0.001 0.001 0.001"/>
     </geometry>
     <material name="silver"/>
@@ -48,5 +48,5 @@
     <origin rpy="0 0 0" xyz="0 0 0"/>
     <geometry>
-      <mesh filename="package://sentry_description/CAD/parts/wheel/wheel.stl" scale="0.001 0.001 0.001"/>
+      <mesh filename="package://sentry_description/CAD/parts/wheel/wheel v3.stl" scale="0.001 0.001 0.001"/>
     </geometry>
   </collision>

Commit message: adding zed camera to model

File: urdf/sentry.xacro (robot description, xacro)
@@ -5,4 +5,5 @@
 <!--<xacro:include filename="$(find sentry_description)/urdf/sentry.trans" />-->
 <xacro:include filename="$(find sentry_description)/urdf/sentry.gazebo" />
+<xacro:include filename="/home/krishan/catkin_ws/src/zed-ros-wrapper/zed_wrapper/urdf/zed_descr.urdf.xacro"/>
 <!--  Base link -->
 <!-- Combine as much bodies as possible into the base_link, this will reduce the complexity of the design -->
@@ -73,25 +74,4 @@
   </collision>
 </link>
-<link name="laser_sensor">
-  <inertial>
-    <!--<origin rpy="0 0 0" xyz="0.16605823931257102 -0.20000099435655025 0.0635739775901992"/>-->
-    <origin rpy="0 0 0" xyz="0 0 0"/>
-    <mass value="0.5"/>
-    <inertia ixx="0.001218" ixy="0.0" ixz="0.0" iyy="0.000635" iyz="0.0" izz="0.000635"/>
-  </inertial>
-  <visual>
-    <origin rpy= "0 0 0" xyz="0 0.22 1.5"/>
-    <geometry>
-      <mesh filename="package://sentry_description/CAD/parts/Lidar/ydlidar_x4 v2.stl" scale="0.001 0.001 0.001"/>
-    </geometry>
-    <material name="silver"/>
-  </visual>
-  <collision>
-    <origin rpy="0 0 0" xyz="0 0 0"/>
-    <geometry>
-      <mesh filename="package://sentry_description/CAD/parts/Lidar/ydlidar_x4 v2.stl" scale="0.001 0.001 0.001"/>
-    </geometry>
-  </collision>
-</link>
 <!-- JOINTS -->
 <!-- The origin of the joint is used as the origin of that component, when positioning above -->
@@ -115,7 +95,7 @@
   <joint_properties damping="1.0" friction="1.0"/>
 </joint>
-<joint name="lidar_joint" type="fixed">
+<joint name="zed_joint" type="fixed">
     <parent link="base_link"/>
-    <child link="laser_sensor"/>s
+    <child link="camera_base_link"/>s
     <origin rpy= "0 0 0" xyz="0 0.22 1.5"/>
 </joint>
