Commit message: Adding mesh

File: urdf/zed_descr.urdf.xacro (robot description, xacro)
@@ -43,20 +43,20 @@
     <link name="$(arg base_frame)">
         <inertial>
-        <origin rpy="0 0 0" xyz="0 0 0"/>
-        <mass value="1"/>
-        <inertia ixx="0.0395416666667" ixy="0" ixz="0" iyy="0.106208333333" iyz="0" izz="0.106208333333"/>
+          <origin rpy="0 0 0" xyz="0 0 0"/>
+          <mass value="1"/>
+          <inertia ixx="0.0395416666667" ixy="0" ixz="0" iyy="0.106208333333" iyz="0" izz="0.106208333333"/>
         </inertial>
         <visual>
-        <origin rpy="0 0 0" xyz="0 0 0"/>
-        <geometry>
-            <mesh filename="package://sentry_description/CAD/parts/base-link/base_link_no wheels v2.stl" scale="0.001 0.001 0.001"/>
-        </geometry>
-        <material name="silver"/>
+          <origin rpy="0 0 0" xyz="0 0 0"/>
+          <geometry>
+              <mesh filename="package://sentry_description/CAD/parts/base-link/base_link_no wheels v2.stl" scale="0.001 0.001 0.001"/>
+          </geometry>
+          <material name="silver"/>
         </visual>
         <collision>
-        <origin rpy="0 0 0" xyz="0 0 0"/>
-        <geometry>
-            <mesh filename="package://sentry_description/CAD/parts/base-link/base_link_no wheels v2.stl" scale="0.001 0.001 0.001"/>
-        </geometry>
+          <origin rpy="0 0 0" xyz="0 0 0"/>
+          <geometry>
+              <mesh filename="package://sentry_description/CAD/parts/base-link/base_link_no wheels v2.stl" scale="0.001 0.001 0.001"/>
+          </geometry>
         </collision>
     </link>
@@ -66,4 +66,5 @@
         <child link="$(arg camera_name)_camera_center"/>
         <origin xyz="$(arg cam_pos_x) $(arg cam_pos_y) $(arg cam_pos_z)" rpy="$(arg cam_roll) $(arg cam_pitch) $(arg cam_yaw)" />
+        <origin rpy="0 0 0" xyz="0 0 0.1"/>
     </joint>
     <link name="$(arg camera_name)_camera_center">
@@ -141,5 +142,5 @@
       <origin rpy="0 0 0" xyz="-0.18650 0 0.114"/>
       <geometry>
-        <mesh filename="package://sentry_description/CAD/parts/wheel/wheel v3.stl" scale="0.001 0.001 0.001"/>
+        <mesh filename="package://sentry_description/CAD/parts/wheel/wheel v7.stl" scale="0.001 0.001 0.001"/>
       </geometry>
       <material name="silver"/>
@@ -148,5 +149,5 @@
       <origin rpy="0 0 0" xyz="0 0 0"/>
       <geometry>
-        <mesh filename="package://sentry_description/CAD/parts/wheel/wheel v3.stl" scale="0.001 0.001 0.001"/>
+        <mesh filename="package://sentry_description/CAD/parts/wheel/wheel v7.stl" scale="0.001 0.001 0.001"/>
       </geometry>
     </collision>
@@ -154,5 +155,5 @@
   <link name="right_wheel">
     <inertial>
-      <!--<origin rpy="0 0 0" xyz="0.16605823931257102 -0.20000099435655025 0.0635739775901992"/>-->
+      <!--<origin rpy="0 0 0" xyz="0.http://wiki.ros.org/rtabmap_ros/Tutorials/SetupOnYourRobot16605823931257102 -0.20000099435655025 0.0635739775901992"/>-->
       <origin rpy="0 0 0" xyz="0 0 0"/>
       <mass value="1"/>
@@ -162,5 +163,5 @@
       <origin rpy="0 0 3.14159" xyz="0.18650 0 0.114"/>
       <geometry>
-        <mesh filename="package://sentry_description/CAD/parts/wheel/wheel v3.stl" scale="0.001 0.001 0.001"/>
+        <mesh filename="package://sentry_description/CAD/parts/wheel/wheel v7.stl" scale="0.001 0.001 0.001"/>
       </geometry>
       <material name="silver"/>
@@ -169,5 +170,5 @@
       <origin rpy="0 0 0" xyz="0 0 0"/>
       <geometry>
-        <mesh filename="package://sentry_description/CAD/parts/wheel/wheel v3.stl" scale="0.001 0.001 0.001"/>
+        <mesh filename="package://sentry_description/CAD/parts/wheel/wheel v7.stl" scale="0.001 0.001 0.001"/>
       </geometry>
     </collision>

Commit message: fixing urdf

File: urdf/zed_descr.urdf.xacro (robot description, xacro)
@@ -1,18 +1,3 @@
 <?xml version="1.0"?>
-<!--
-Copyright (c) 2020, STEREOLABS.
-All rights reserved.
-THIS SOFTWARE IS PROVIDED BY THE COPYRIGHT HOLDERS AND CONTRIBUTORS
-"AS IS" AND ANY EXPRESS OR IMPLIED WARRANTIES, INCLUDING, BUT NOT
-LIMITED TO, THE IMPLIED WARRANTIES OF MERCHANTABILITY AND FITNESS FOR
-A PARTICULAR PURPOSE ARE DISCLAIMED. IN NO EVENT SHALL THE COPYRIGHT
-OWNER OR CONTRIBUTORS BE LIABLE FOR ANY DIRECT, INDIRECT, INCIDENTAL,
-SPECIAL, EXEMPLARY, OR CONSEQUENTIAL DAMAGES (INCLUDING, BUT NOT
-LIMITED TO, PROCUREMENT OF SUBSTITUTE GOODS OR SERVICES; LOSS OF USE,
-DATA, OR PROFITS; OR BUSINESS INTERRUPTION) HOWEVER CAUSED AND ON ANY
-THEORY OF LIABILITY, WHETHER IN CONTRACT, STRICT LIABILITY, OR TORT
-(INCLUDING NEGLIGENCE OR OTHERWISE) ARISING IN ANY WAY OUT OF THE USE
-OF THIS SOFTWARE, EVEN IF ADVISED OF THE POSSIBILITY OF SUCH DAMAGE.
--->
 <robot name="stereolabs_camera" xmlns:xacro="http://ros.org/wiki/xacro">
 <!-- Includes -->
@@ -65,6 +50,6 @@
         <parent link="$(arg base_frame)"/>
         <child link="$(arg camera_name)_camera_center"/>
-        <origin xyz="$(arg cam_pos_x) $(arg cam_pos_y) $(arg cam_pos_z)" rpy="$(arg cam_roll) $(arg cam_pitch) $(arg cam_yaw)" />
-        <origin rpy="0 0 0" xyz="0 0 0.1"/>
+        <!--<origin xyz="$(arg cam_pos_x) $(arg cam_pos_y) $(arg cam_pos_z)" rpy="$(arg cam_roll) $(arg cam_pitch) $(arg cam_yaw)" />-->
+        <origin rpy="0 0 0" xyz="0 0 1.5"/>
     </joint>
     <link name="$(arg camera_name)_camera_center">
@@ -140,5 +125,5 @@
     </inertial>
     <visual>
-      <origin rpy="0 0 0" xyz="-0.18650 0 0.114"/>
+      <origin rpy="0 0 0" xyz="0 0 0"/>
       <geometry>
         <mesh filename="package://sentry_description/CAD/parts/wheel/wheel v7.stl" scale="0.001 0.001 0.001"/>
@@ -161,5 +146,5 @@
     </inertial>
     <visual>
-      <origin rpy="0 0 3.14159" xyz="0.18650 0 0.114"/>
+      <origin rpy="3.14159 0 0" xyz="0 0 0"/>
       <geometry>
         <mesh filename="package://sentry_description/CAD/parts/wheel/wheel v7.stl" scale="0.001 0.001 0.001"/>
@@ -175,5 +160,5 @@
   </link>
   <joint name="left_wheel_joint" type="continuous">
-    <origin rpy="0 0 0" xyz="-0.18650 0 0.114"/>
+    <origin rpy="0 0 3.14159" xyz="0 0 0"/>
     <parent link="$(arg base_frame)" />
     <child link="left_wheel"/>
@@ -182,8 +167,9 @@
     <joint_properties damping="1.0" friction="1.0"/>
   </joint>
-  <!-- Joint between right wheel and Base Link -->
+  <!-- Joint between_ws$ sudo apt-get install ros-melodic-joint-state-pubisher
+[sudo] password for krishan: n right wheel and Base Link -->
   <joint name="right_wheel_joint" type="continuous">
   <!-- yaw set to 3.14159 to flip the wheel and align it properly-->
-    <origin rpy="0 0 3.14159" xyz="0.18650 0 0.114"/>
+    <origin rpy="0 0 3.14159" xyz="0 0 0"/>
     <parent link="$(arg base_frame)" />
     <child link="right_wheel"/>

Commit message: adding joint

File: urdf/zed_descr.urdf.xacro (robot description, xacro)
@@ -160,5 +160,5 @@
   </link>
   <joint name="left_wheel_joint" type="continuous">
-    <origin rpy="0 0 3.14159" xyz="0 0 0"/>
+    <origin rpy="0 0 0" xyz="0 -0.5 0"/>
     <parent link="$(arg base_frame)" />
     <child link="left_wheel"/>
@@ -167,9 +167,7 @@
     <joint_properties damping="1.0" friction="1.0"/>
   </joint>
-  <!-- Joint between_ws$ sudo apt-get install ros-melodic-joint-state-pubisher
-[sudo] password for krishan: n right wheel and Base Link -->
   <joint name="right_wheel_joint" type="continuous">
   <!-- yaw set to 3.14159 to flip the wheel and align it properly-->
-    <origin rpy="0 0 3.14159" xyz="0 0 0"/>
+    <origin rpy="0 -3.14159 0" xyz="0 0.5 0"/>
     <parent link="$(arg base_frame)" />
     <child link="right_wheel"/>

Commit message: adding tilt

File: urdf/zed_descr.urdf.xacro (robot description, xacro)
@@ -51,5 +51,5 @@
         <child link="$(arg camera_name)_camera_center"/>
         <!--<origin xyz="$(arg cam_pos_x) $(arg cam_pos_y) $(arg cam_pos_z)" rpy="$(arg cam_roll) $(arg cam_pitch) $(arg cam_yaw)" />-->
-        <origin rpy="0 1.5708 1.5708" xyz="0 0 0"/>
+        <origin rpy="0 1.5708 1.5708" xyz="3.141592654 0 0"/>
     </joint>
     <link name="$(arg camera_name)_camera_center">
@@ -66,5 +66,5 @@
         <parent link="$(arg camera_name)_camera_center"/>
         <child link="$(arg camera_name)_left_camera_frame"/>
-        <origin xyz="0 ${baseline/2} 0" rpy="0 0 0" />
+        <origin xyz="0 ${baseline/2} 0" rpy="3.141592654 0 0" />
     </joint>
     <link name="$(arg camera_name)_left_camera_frame" />
@@ -93,5 +93,5 @@
             <parent link="$(arg camera_name)_camera_center"/>
             <child link="$(arg camera_name)_mag_link"/>
-            <origin xyz="0 0 0" rpy="0 0 0" />
+            <origin xyz="0 0 0" rpy="3.141592654 0 0" />
         </joint>
         <link name="$(arg camera_name)_mag_link" />
@@ -99,5 +99,5 @@
             <parent link="$(arg camera_name)_camera_center"/>
             <child link="$(arg camera_name)_baro_link"/>
-            <origin xyz="0 0 0" rpy="0 0 0" />
+            <origin xyz="0 0 0" rpy="3.141592654 0 0" />
         </joint>
         <link name="$(arg camera_name)_baro_link" />
@@ -105,5 +105,5 @@
             <parent link="$(arg camera_name)_left_camera_frame"/>
             <child link="$(arg camera_name)_temp_left_link"/>
-            <origin xyz="0 0 0" rpy="0 0 0" />
+            <origin xyz="0 0 0" rpy="3.141592654 0 0" />
         </joint>
         <link name="$(arg camera_name)_temp_left_link" />
@@ -111,5 +111,5 @@
             <parent link="$(arg camera_name)_right_camera_frame"/>
             <child link="$(arg camera_name)_temp_right_link"/>
-            <origin xyz="0 0 0" rpy="0 0 0" />
+            <origin xyz="0 0 0" rpy="3.141592654 0 0" />
         </joint>
         <link name="$(arg camera_name)_temp_right_link" />

Commit message: changing dimensions

File: urdf/zed_descr.urdf.xacro (robot description, xacro)
@@ -161,5 +161,5 @@
    <!--Wheel Joints-->
   <joint name="left_wheel_joint" type="continuous">
-    <origin rpy="0 0 0" xyz="0 -0.1 -0.5"/>
+    <origin rpy="0 0 0" xyz="-0.25 0 0"/>
     <parent link="$(arg base_frame)" />
     <child link="left_wheel"/>
@@ -170,5 +170,5 @@
   <joint name="right_wheel_joint" type="continuous">
   <!-- yaw set to 3.14159 to flip the wheel and align it properly-->
-    <origin rpy="0 -0 0" xyz="0 0.1 -0.05"/>
+    <origin rpy="0 0 0" xyz="0.25 0 0"/>
     <parent link="$(arg base_frame)" />
     <child link="right_wheel"/>

Commit message: changing map offset

File: urdf/zed_descr.urdf.xacro (robot description, xacro)
@@ -51,5 +51,5 @@
         <child link="$(arg camera_name)_camera_center"/>
         <!--<origin xyz="$(arg cam_pos_x) $(arg cam_pos_y) $(arg cam_pos_z)" rpy="$(arg cam_roll) $(arg cam_pitch) $(arg cam_yaw)" />-->
-        <origin rpy="0 1.5708 1.5708" xyz="3.141592654 0 0"/>
+        <origin rpy="0 0 0" xyz="3.141592654 0 0"/>
     </joint>
     <link name="$(arg camera_name)_camera_center">
@@ -161,5 +161,5 @@
    <!--Wheel Joints-->
   <joint name="left_wheel_joint" type="continuous">
-    <origin rpy="0 0 0" xyz="-0.25 0 0"/>
+    <origin rpy="0 0 0" xyz="-0.2 0 0"/>
     <parent link="$(arg base_frame)" />
     <child link="left_wheel"/>
@@ -170,5 +170,5 @@
   <joint name="right_wheel_joint" type="continuous">
   <!-- yaw set to 3.14159 to flip the wheel and align it properly-->
-    <origin rpy="0 0 0" xyz="0.25 0 0"/>
+    <origin rpy="0 0 0" xyz="0.2 0 0"/>
     <parent link="$(arg base_frame)" />
     <child link="right_wheel"/>

Commit message: Updates

File: urdf/zed_descr.urdf.xacro (robot description, xacro)
@@ -7,7 +7,7 @@
     <xacro:arg name="camera_model"  default="zed" />
     <xacro:arg name="base_frame"    default="base_link" />
-    <xacro:arg name="cam_pos_x"     default="0.22" />
+    <xacro:arg name="cam_pos_x"     default="-0.35" />
     <xacro:arg name="cam_pos_y"     default="0.0" />
-    <xacro:arg name="cam_pos_z"     default="1.5768" />
+    <xacro:arg name="cam_pos_z"     default="0.5" />
     <xacro:arg name="cam_roll"      default="0.0" />
     <xacro:arg name="cam_pitch"     default="0.0" />
@@ -50,6 +50,5 @@
         <parent link="$(arg base_frame)"/>
         <child link="$(arg camera_name)_camera_center"/>
-        <!--<origin xyz="$(arg cam_pos_x) $(arg cam_pos_y) $(arg cam_pos_z)" rpy="$(arg cam_roll) $(arg cam_pitch) $(arg cam_yaw)" />-->
-        <origin rpy="0 0 0" xyz="3.141592654 0 0"/>
+        <origin xyz="$(arg cam_pos_x) $(arg cam_pos_y) $(arg cam_pos_z)" rpy="$(arg cam_roll) $(arg cam_pitch) $(arg cam_yaw)" />
     </joint>
     <link name="$(arg camera_name)_camera_center">
